File: bipop_power_supply.brd (EAGLE design)
At the start: 82.5 x 70.8 mm, 28 parts, among them IC1 LM1117MP-3.3, IC2 LM1117MP-5.0, X2 MSTBA6

Commit message: minor changes in PoSup PCB design
Parts:
- moved D6 1.27 mm to (21.6, 64.8)
- moved D2 1.27 mm to (21.6, 57.1)
- moved C8 1.27 mm to (20.3, 30.5)
- moved D5 1.27 mm to (20.3, 50.8)
- moved D1 1.27 mm to (20.3, 48.3)
Routing:
- net MM: track 61.4 -> 74.4 mm
- net 12_OUT: track 66.5 -> 70.3 mm
- net 3_OUT: track 85.9 -> 82.4 mm
- net VCC_3V3: track 118.7 -> 121.6 mm
- net GND: track 203.1 -> 205.8 mm
- net N$16: track 9.66 -> 7.86 mm
- net 5_OUT: track 54.7 -> 56.0 mm
- net N$3: track 39.7 -> 40.9 mm
- net 12_IN: track 20.0 -> 20.5 mm
